Commit message: Publish the camera in REP-145 optical frames

File: workspace/src/g1_description/urdf/g1_arm_sdk.urdf.xacro (robot description, xacro)
@@ -3,4 +3,22 @@
   <!-- Verbatim upstream description; xacro:include discards <robot> wrapper. -->
   <xacro:include filename="g1_29dof_with_hand_rev_1_0.urdf"/>
+  <!-- REP-145 optical frames. The vendored URDF stops at d435_link, which is a body frame
+       (x forward, y left, z up); every ROS depth consumer, rviz's DepthCloud included,
+       assumes the optical convention (z forward, x right, y down). Publishing a depth
+       image in the body frame projects it rotated 90 degrees, which looks like a broken
+       sensor rather than a wrong frame. Added here rather than in the vendored file so
+       that stays verbatim. -->
+  <link name="camera_depth_optical_frame"/>
+  <joint name="camera_depth_optical_joint" type="fixed">
+    <parent link="d435_link"/>
+    <child link="camera_depth_optical_frame"/>
+    <origin xyz="0 0 0" rpy="-1.5707963267948966 0 -1.5707963267948966"/>
+  </joint>
+  <link name="camera_color_optical_frame"/>
+  <joint name="camera_color_optical_joint" type="fixed">
+    <parent link="d435_link"/>
+    <child link="camera_color_optical_frame"/>
+    <origin xyz="0 0 0" rpy="-1.5707963267948966 0 -1.5707963267948966"/>
+  </joint>
   <!-- Load tunable YAML for ROS 2 control parameters. -->
   <xacro:property name="arm_sdk_params" value="${xacro.load_yaml('../config/arm_sdk_params.yaml')}"/>

Commit message: Give the depth camera and LiDAR visual bodies

File: workspace/src/g1_description/urdf/g1_arm_sdk.urdf.xacro (robot description, xacro)
@@ -23,4 +23,46 @@
     <child link="camera_color_optical_frame"/>
     <origin xyz="0 0 0" rpy="-1.5707963267948966 0 -1.5707963267948966"/>
+  </joint>
+  <!-- Sensor bodies. The vendored URDF leaves d435_link and mid360_link as EMPTY links, so both
+       sensors are invisible in RViz and it is impossible to see where either is pointing.
+       Attached as child links rather than by editing those links, for the same reason the
+       optical frames above are: the vendored file stays byte-for-byte diffable against
+       Unitree's.
+       VISUAL ONLY, deliberately. Collision geometry here would be swept into MoveIt's
+       self-filter and its planning scene, so a mis-sized box would silently either carve a hole
+       in the octomap or block plans near the head. These exist to be looked at, nothing more.
+       See g1_moveit_config/config/sensors_3d.yaml for what the sensors actually feed. -->
+  <link name="d435_visual">
+    <visual>
+      <!-- Intel's own placement from realsense2_description's _d435.urdf.xacro: the mesh origin
+           sits at the front plate between the two infrared cameras, so it needs this offset and
+           rotation to line up with the link. Values are
+           d435_zero_depth_to_glass + d435_glass_to_front, and -d435_cam_depth_py. -->
+      <origin xyz="0.0043 -0.0175 0" rpy="1.5707963267948966 0 1.5707963267948966"/>
+      <geometry>
+        <mesh filename="package://realsense2_description/meshes/d435.dae"/>
+      </geometry>
+    </visual>
+  </link>
+  <joint name="d435_visual_joint" type="fixed">
+    <parent link="d435_link"/>
+    <child link="d435_visual"/>
+  </joint>
+  <link name="mid360_visual">
+    <visual>
+      <!-- Livox ship no ROS description package, so this is a primitive from the published
+           MID360 dimensions (65 x 65 x 60 mm) rather than a mesh. It marks where the LiDAR is
+           and roughly how big; do not read anything finer off it. -->
+      <geometry>
+        <cylinder radius="0.0325" length="0.060"/>
+      </geometry>
+      <material name="dark_grey">
+        <color rgba="0.15 0.15 0.15 1.0"/>
+      </material>
+    </visual>
+  </link>
+  <joint name="mid360_visual_joint" type="fixed">
+    <parent link="mid360_link"/>
+    <child link="mid360_visual"/>
   </joint>
   <!-- Load tunable YAML for ROS 2 control parameters. -->

Commit message: Give the hands a ros2_control component each

File: workspace/src/g1_description/urdf/g1_arm_sdk.urdf.xacro (robot description, xacro)
@@ -105,3 +105,43 @@
     <xacro:g1_arm_joint name="right_wrist_yaw_joint"/>
   </ros2_control>
+  <xacro:property name="dex3_params" value="${xacro.load_yaml('../config/dex3_params.yaml')}"/>
+  <xacro:macro name="g1_hand_joint" params="name">
+    <joint name="${name}">
+      <command_interface name="position"/>
+      <state_interface name="position"/>
+      <state_interface name="velocity"/>
+      <state_interface name="effort"/>
+      <param name="min">${dex3_params.joints[name].min}</param>
+      <param name="max">${dex3_params.joints[name].max}</param>
+    </joint>
+  </xacro:macro>
+  <!-- One component per hand. The Dex3 is a separate device on its own DDS topics with its
+       own authority (docs/CONTROL_MODES.md), so it is neither folded into G1ArmSdkSystem nor
+       shared between the two hands: a fault on one hand must not take the arms or the other
+       hand down with it.
+       Joint order is the Dex3 wire order and G1Dex3System refuses to init if it is disturbed,
+       because HandCmd.motor_cmd is a positional array and a reordered list would close the
+       wrong fingers. -->
+  <xacro:macro name="g1_dex3_hand" params="side">
+    <ros2_control name="G1Dex3System${'Left' if side == 'left' else 'Right'}" type="system">
+      <hardware>
+        <plugin>g1_hand_interface/G1Dex3System</plugin>
+        <param name="side">${side}</param>
+        <param name="kp">${dex3_params.system.kp}</param>
+        <param name="kd">${dex3_params.system.kd}</param>
+        <param name="command_publish_rate">${dex3_params.system.command_publish_rate}</param>
+        <param name="max_joint_velocity_rad_s">${dex3_params.system.max_joint_velocity_rad_s}</param>
+        <param name="state_timeout_ms">${dex3_params.system.state_timeout_ms}</param>
+      </hardware>
+      <xacro:g1_hand_joint name="${side}_hand_thumb_0_joint"/>
+      <xacro:g1_hand_joint name="${side}_hand_thumb_1_joint"/>
+      <xacro:g1_hand_joint name="${side}_hand_thumb_2_joint"/>
+      <xacro:g1_hand_joint name="${side}_hand_middle_0_joint"/>
+      <xacro:g1_hand_joint name="${side}_hand_middle_1_joint"/>
+      <xacro:g1_hand_joint name="${side}_hand_index_0_joint"/>
+      <xacro:g1_hand_joint name="${side}_hand_index_1_joint"/>
+    </ros2_control>
+  </xacro:macro>
+  <xacro:g1_dex3_hand side="left"/>
+  <xacro:g1_dex3_hand side="right"/>
 </robot>

Commit message: Plan to a grasp frame in the URDF instead of a palm offset

File: workspace/src/g1_description/urdf/g1_arm_sdk.urdf.xacro (robot description, xacro)
@@ -145,3 +145,30 @@
   <xacro:g1_dex3_hand side="left"/>
   <xacro:g1_dex3_hand side="right"/>
+  <!-- Where the hand actually closes, as a frame rather than a number in a config file.
+       The palm link's origin is NOT the point the fingers grip at, and the difference is large
+       enough to matter: at the SRDF's `closed` posture the thumb tip lands at palm
+       (-0.030, +0.020, +0.017) and the middle and index tips at (+0.050, +0.068, -/+0.029), so
+       what the hand encloses sits well forward of the origin and mostly to one side of it.
+       Planning to the palm origin puts the object through the fingers.
+       A frame, not a parameter, for three reasons. It is visible in RViz, so being wrong is
+       something you can see rather than infer from a failed plan. MoveIt can be given a pose
+       goal for it directly, so no code does offset arithmetic. And it is a property of the
+       Dex3's own geometry, identical on the real hand, so it belongs in the description
+       alongside everything else the URDF says about the hand.
+       Orientation matches the palm, so a caller still chooses how to hold the hand; only the
+       position is corrected. The two hands mirror, which is why y and z flip.
+       The value is derived from the URDF's own finger chain and is the piece most worth
+       re-measuring against the real hand: the fingertip offset past the last joint is
+       estimated from link inertials rather than from the meshes. Being a frame, checking it
+       is a matter of looking at it in RViz. -->
+  <xacro:macro name="g1_grasp_frame" params="side mirror">
+    <link name="${side}_hand_grasp_frame"/>
+    <joint name="${side}_hand_grasp_frame_joint" type="fixed">
+      <parent link="${side}_hand_palm_link"/>
+      <child link="${side}_hand_grasp_frame"/>
+      <origin xyz="0.010 ${mirror * 0.044} ${mirror * 0.009}" rpy="0 0 0"/>
+    </joint>
+  </xacro:macro>
+  <xacro:g1_grasp_frame side="left" mirror="-1"/>
+  <xacro:g1_grasp_frame side="right" mirror="1"/>
 </robot>

Commit message: Wire FAST-LIO end to end: configs, launch, converter, mid360_imu frame

File: workspace/src/g1_description/urdf/g1_arm_sdk.urdf.xacro (robot description, xacro)
@@ -65,4 +65,14 @@
     <parent link="mid360_link"/>
     <child link="mid360_visual"/>
+  </joint>
+  <!-- The Mid360's built-in IMU, which is the frame FAST-LIO's odometry reports ("body").
+       Livox publish the LIDAR-in-IMU offset [-0.011, -0.02329, 0.04412]; this joint is its
+       inverse, because here the parent is the lidar frame the cloud arrives in. Rotation is
+       identity: both sensors sit in one housing and flip together with the mount. -->
+  <link name="mid360_imu"/>
+  <joint name="mid360_imu_joint" type="fixed">
+    <parent link="mid360_link"/>
+    <child link="mid360_imu"/>
+    <origin xyz="0.011 0.02329 -0.04412" rpy="0 0 0"/>
   </joint>
   <!-- Load tunable YAML for ROS 2 control parameters. -->

Commit message: Share the body, frames and hands between both stack descriptions

File: workspace/src/g1_description/urdf/g1_arm_sdk.urdf.xacro (robot description, xacro)
@@ -1,79 +1,7 @@
 <?xml version="1.0"?>
 <robot xmlns:xacro="http://www.ros.org/wiki/xacro" name="g1_29dof_with_hand_rev_1_0">
-  <!-- Upstream description, with one mechanical edit: mesh paths were changed from relative
-       ("meshes/x.STL") to package:// so RViz can resolve them. See g1_description/README.md.
-       Everything else is byte-for-byte upstream, CRLF included, so it stays diffable against
-       Unitree's file. xacro:include discards the <robot> wrapper. -->
-  <xacro:include filename="g1_29dof_with_hand_rev_1_0.urdf"/>
-  <!-- REP-145 optical frames. The vendored URDF stops at d435_link, which is a body frame
-       (x forward, y left, z up); every ROS depth consumer, rviz's DepthCloud included,
-       assumes the optical convention (z forward, x right, y down). Publishing a depth
-       image in the body frame projects it rotated 90 degrees, which looks like a broken
-       sensor rather than a wrong frame. Added here rather than in the vendored file, which
-       is kept as close to upstream as possible. -->
-  <link name="camera_depth_optical_frame"/>
-  <joint name="camera_depth_optical_joint" type="fixed">
-    <parent link="d435_link"/>
-    <child link="camera_depth_optical_frame"/>
-    <origin xyz="0 0 0" rpy="-1.5707963267948966 0 -1.5707963267948966"/>
-  </joint>
-  <link name="camera_color_optical_frame"/>
-  <joint name="camera_color_optical_joint" type="fixed">
-    <parent link="d435_link"/>
-    <child link="camera_color_optical_frame"/>
-    <origin xyz="0 0 0" rpy="-1.5707963267948966 0 -1.5707963267948966"/>
-  </joint>
-  <!-- Sensor bodies. The vendored URDF leaves d435_link and mid360_link as empty links, so both
-       sensors are invisible in RViz and it is impossible to see where either is pointing.
-       Attached as child links rather than by editing those links, for the same reason the
-       optical frames above are: the vendored file stays byte-for-byte diffable against
-       Unitree's.
-       VISUAL ONLY, deliberately. Collision geometry here would be swept into MoveIt's
-       self-filter and its planning scene, so a mis-sized box would silently either carve a hole
-       in the octomap or block plans near the head. These exist to be looked at, nothing more.
-       See g1_moveit_config/config/sensors_3d.yaml for what the sensors actually feed. -->
-  <link name="d435_visual">
-    <visual>
-      <!-- Intel's own placement from realsense2_description's _d435.urdf.xacro: the mesh origin
-           sits at the front plate between the two infrared cameras, so it needs this offset and
-           rotation to line up with the link. Values are
-           d435_zero_depth_to_glass + d435_glass_to_front, and -d435_cam_depth_py. -->
-      <origin xyz="0.0043 -0.0175 0" rpy="1.5707963267948966 0 1.5707963267948966"/>
-      <geometry>
-        <mesh filename="package://realsense2_description/meshes/d435.dae"/>
-      </geometry>
-    </visual>
-  </link>
-  <joint name="d435_visual_joint" type="fixed">
-    <parent link="d435_link"/>
-    <child link="d435_visual"/>
-  </joint>
-  <link name="mid360_visual">
-    <visual>
-      <!-- Livox ship no ROS description package, so this is a primitive from the published
-           MID360 dimensions (65 x 65 x 60 mm) rather than a mesh. It marks where the LiDAR is
-           and roughly how big; do not read anything finer off it. -->
-      <geometry>
-        <cylinder radius="0.0325" length="0.060"/>
-      </geometry>
-      <material name="dark_grey">
-        <color rgba="0.15 0.15 0.15 1.0"/>
-      </material>
-    </visual>
-  </link>
-  <joint name="mid360_visual_joint" type="fixed">
-    <parent link="mid360_link"/>
-    <child link="mid360_visual"/>
-  </joint>
-  <!-- The Mid360's built-in IMU, which is the frame FAST-LIO's odometry reports ("body").
-       Livox publish the LIDAR-in-IMU offset [-0.011, -0.02329, 0.04412]; this joint is its
-       inverse, because here the parent is the lidar frame the cloud arrives in. Rotation is
-       identity: both sensors sit in one housing and flip together with the mount. -->
-  <link name="mid360_imu"/>
-  <joint name="mid360_imu_joint" type="fixed">
-    <parent link="mid360_link"/>
-    <child link="mid360_imu"/>
-    <origin xyz="0.011 0.02329 -0.04412" rpy="0 0 0"/>
-  </joint>
+  <!-- The body, the frames and both hands. Shared with g1_lowcmd.urdf.xacro so a grasp frame or
+       a sensor extrinsic cannot drift between the two stacks. -->
+  <xacro:include filename="g1_common.xacro"/>
   <!-- Load tunable YAML for ROS 2 control parameters. -->
   <xacro:property name="arm_sdk_params" value="${xacro.load_yaml('../config/arm_sdk_params.yaml')}"/>
@@ -119,71 +47,3 @@
     <xacro:g1_arm_joint name="right_wrist_yaw_joint"/>
   </ros2_control>
-  <xacro:property name="dex3_params" value="${xacro.load_yaml('../config/dex3_params.yaml')}"/>
-  <xacro:macro name="g1_hand_joint" params="name">
-    <joint name="${name}">
-      <command_interface name="position"/>
-      <state_interface name="position"/>
-      <state_interface name="velocity"/>
-      <state_interface name="effort"/>
-      <param name="min">${dex3_params.joints[name].min}</param>
-      <param name="max">${dex3_params.joints[name].max}</param>
-    </joint>
-  </xacro:macro>
-  <!-- One component per hand. The Dex3 is a separate device on its own DDS topics with its
-       own authority, so it is neither folded into G1ArmSdkSystem nor
-       shared between the two hands: a fault on one hand must not take the arms or the other
-       hand down with it.
-       Joint order is the Dex3 wire order and G1Dex3System refuses to init if it is disturbed,
-       because HandCmd.motor_cmd is a positional array and a reordered list would close the
-       wrong fingers. -->
-  <xacro:macro name="g1_dex3_hand" params="side">
-    <ros2_control name="G1Dex3System${'Left' if side == 'left' else 'Right'}" type="system">
-      <hardware>
-        <plugin>g1_hand_interface/G1Dex3System</plugin>
-        <param name="side">${side}</param>
-        <param name="kp">${dex3_params.system.kp}</param>
-        <param name="kd">${dex3_params.system.kd}</param>
-        <param name="command_publish_rate">${dex3_params.system.command_publish_rate}</param>
-        <param name="max_joint_velocity_rad_s">${dex3_params.system.max_joint_velocity_rad_s}</param>
-        <param name="state_timeout_ms">${dex3_params.system.state_timeout_ms}</param>
-        <param name="state_topic">${dex3_params.system.state_topic_prefix}${side}${dex3_params.system.state_topic_suffix}</param>
-      </hardware>
-      <xacro:g1_hand_joint name="${side}_hand_thumb_0_joint"/>
-      <xacro:g1_hand_joint name="${side}_hand_thumb_1_joint"/>
-      <xacro:g1_hand_joint name="${side}_hand_thumb_2_joint"/>
-      <xacro:g1_hand_joint name="${side}_hand_middle_0_joint"/>
-      <xacro:g1_hand_joint name="${side}_hand_middle_1_joint"/>
-      <xacro:g1_hand_joint name="${side}_hand_index_0_joint"/>
-      <xacro:g1_hand_joint name="${side}_hand_index_1_joint"/>
-    </ros2_control>
-  </xacro:macro>
-  <xacro:g1_dex3_hand side="left"/>
-  <xacro:g1_dex3_hand side="right"/>
-  <!-- Where the hand actually closes, as a frame rather than a number in a config file.
-       The palm link's origin is not the point the fingers grip at, and the difference is large
-       enough to matter: at the SRDF's `closed` posture the thumb tip lands at palm
-       (-0.030, +0.020, +0.017) and the middle and index tips at (+0.050, +0.068, -/+0.029), so
-       what the hand encloses sits well forward of the origin and mostly to one side of it.
-       Planning to the palm origin puts the object through the fingers.
-       A frame, not a parameter, for three reasons. It is visible in RViz, so being wrong is
-       something you can see rather than infer from a failed plan. MoveIt can be given a pose
-       goal for it directly, so no code does offset arithmetic. And it is a property of the
-       Dex3's own geometry, identical on the real hand, so it belongs in the description
-       alongside everything else the URDF says about the hand.
-       Orientation matches the palm, so a caller still chooses how to hold the hand; only the
-       position is corrected. The two hands mirror, which is why y and z flip.
-       The value is derived from the URDF's own finger chain and is the piece most worth
-       re-measuring against the real hand: the fingertip offset past the last joint is
-       estimated from link inertials rather than from the meshes. Being a frame, checking it
-       is a matter of looking at it in RViz. -->
-  <xacro:macro name="g1_grasp_frame" params="side mirror">
-    <link name="${side}_hand_grasp_frame"/>
-    <joint name="${side}_hand_grasp_frame_joint" type="fixed">
-      <parent link="${side}_hand_palm_link"/>
-      <child link="${side}_hand_grasp_frame"/>
-      <origin xyz="0.010 ${mirror * 0.044} ${mirror * 0.009}" rpy="0 0 0"/>
-    </joint>
-  </xacro:macro>
-  <xacro:g1_grasp_frame side="left" mirror="-1"/>
-  <xacro:g1_grasp_frame side="right" mirror="1"/>
 </robot>

File: workspace/src/g1_description/urdf/g1_lowcmd.urdf.xacro (robot description, xacro)
@@ -3,6 +3,8 @@
   <!-- Whole-body variant: the 29 body motors are owned by G1LowCmdSystem over rt/lowcmd, with no
        onboard balance running underneath. g1_arm_sdk.urdf.xacro is the blended-arm variant and
-       stays until PR 6 retires it. Only one of the two may be loaded at a time. -->
-  <xacro:include filename="g1_29dof_with_hand_rev_1_0.urdf"/>
+       stays until PR 6 retires it. Only one of the two may be loaded at a time.
+       g1_common.xacro brings the body, the sensor and grasp frames, and both Dex3 components:
+       everything that is identical whichever interface owns the motors. -->
+  <xacro:include filename="g1_common.xacro"/>
   <xacro:property name="lowcmd" value="${xacro.load_yaml('../config/lowcmd_params.yaml')}"/>
   <xacro:macro name="g1_lowcmd_joint" params="name">
