Commit message: Put the grasp frame where the hand actually closes

File: workspace/src/g1_description/urdf/g1_common.xacro (robot description, xacro)
@@ -127,8 +127,5 @@
   <!-- Where the hand actually closes, as a frame rather than a number in a config file.
        The palm link's origin is not the point the fingers grip at, and the difference is large
-       enough to matter: at the SRDF's `closed` posture the thumb tip lands at palm
-       (-0.030, +0.020, +0.017) and the middle and index tips at (+0.050, +0.068, -/+0.029), so
-       what the hand encloses sits well forward of the origin and mostly to one side of it.
-       Planning to the palm origin puts the object through the fingers.
+       enough to matter: planning to the palm origin puts the object through the fingers.
        A frame, not a parameter, for three reasons. It is visible in RViz, so being wrong is
        something you can see rather than infer from a failed plan. MoveIt can be given a pose
@@ -137,9 +134,14 @@
        alongside everything else the URDF says about the hand.
        Orientation matches the palm, so a caller still chooses how to hold the hand; only the
-       position is corrected. The two hands mirror, which is why y and z flip.
-       The value is derived from the URDF's own finger chain and is the piece most worth
-       re-measuring against the real hand: the fingertip offset past the last joint is
-       estimated from link inertials rather than from the meshes. Being a frame, checking it
-       is a matter of looking at it in RViz. -->
+       position is corrected. The two hands mirror, which is why y flips.
+       x = 0.090 is bounded on both sides, measured against the finger collision capsules in
+       MuJoCo rather than estimated. The thumb's own surface sits at palm x = 0.046 at
+       `pinch_ready`, so anything nearer than that is in the space the hand descends through;
+       and the thumb only swings out to x = 0.091 at `closed`, so anything further and it never
+       reaches the object at all. Between them this frame takes objects 20 to 75 mm across.
+       y = 0.050 is where the fingers and thumb meet, and it is also what fixes how tall an
+       object has to be: the hand hangs 113 mm below the palm even with the thumb retracted, so
+       63 mm below this frame, and an object shorter than that gets the thumb on the table
+       instead. See g1_manipulation's grasp_depth_below_top_m and min_grip_height_m. -->
   <xacro:macro name="g1_grasp_frame" params="side mirror">
     <link name="${side}_hand_grasp_frame"/>
@@ -147,5 +149,5 @@
       <parent link="${side}_hand_palm_link"/>
       <child link="${side}_hand_grasp_frame"/>
-      <origin xyz="0.010 ${mirror * 0.044} ${mirror * 0.009}" rpy="0 0 0"/>
+      <origin xyz="0.090 ${mirror * 0.050} 0" rpy="0 0 0"/>
     </joint>
   </xacro:macro>

Commit message: Put the grasp frame where a held object actually sits

File: workspace/src/g1_description/urdf/g1_common.xacro (robot description, xacro)
@@ -140,8 +140,19 @@
        and the thumb only swings out to x = 0.091 at `closed`, so anything further and it never
        reaches the object at all. Between them this frame takes objects 20 to 75 mm across.
-       y = 0.050 is where the fingers and thumb meet, and it is also what fixes how tall an
-       object has to be: the hand hangs 113 mm below the palm even with the thumb retracted, so
-       63 mm below this frame, and an object shorter than that gets the thumb on the table
-       instead. See g1_manipulation's grasp_depth_below_top_m and min_grip_height_m. -->
+       y = 0.085 is where a held object actually ends up, which is not where the thumb and
+       finger LINK ORIGINS meet. That midpoint is y = 0.050 and this frame used to sit on it,
+       but the collision capsules run 50 to 62 mm out along each link, so the volume the hand
+       closes on is much further out than its joint origins suggest.
+       Measured rather than derived: with ground truth for the block and TF for the palm, a
+       block held through a carry sits at palm (0.086, 0.089, 0.002) while the frame claimed
+       (0.090, 0.050, 0.000). x and z agree to 4 mm and y is out by 39 mm, which is a frame
+       error along the closing axis and not scatter. Every finger was at or near its 1.4 N.m
+       torque clamp at the time, so the hand was gripping hard, just 39 mm too far out, where
+       the object levers itself free: it rotated from 14 to 33 degrees during the lift and slid
+       19 mm while the hand rose 184 mm.
+       It also fixes how tall an object has to be: the hand hangs 113 mm below the palm even
+       with the thumb retracted, so 28 mm below this frame, and an object shorter than that gets
+       the thumb on the table instead. See g1_manipulation's grasp_depth_below_top_m and
+       min_grip_height_m. -->
   <xacro:macro name="g1_grasp_frame" params="side mirror">
     <link name="${side}_hand_grasp_frame"/>
@@ -149,5 +160,5 @@
       <parent link="${side}_hand_palm_link"/>
       <child link="${side}_hand_grasp_frame"/>
-      <origin xyz="0.090 ${mirror * 0.050} 0" rpy="0 0 0"/>
+      <origin xyz="0.090 ${mirror * 0.085} 0" rpy="0 0 0"/>
     </joint>
   </xacro:macro>

Commit message: Put the grasp frame back where the descent can reach

File: workspace/src/g1_description/urdf/g1_common.xacro (robot description, xacro)
@@ -140,19 +140,24 @@
        and the thumb only swings out to x = 0.091 at `closed`, so anything further and it never
        reaches the object at all. Between them this frame takes objects 20 to 75 mm across.
-       y = 0.085 is where a held object actually ends up, which is not where the thumb and
-       finger LINK ORIGINS meet. That midpoint is y = 0.050 and this frame used to sit on it,
-       but the collision capsules run 50 to 62 mm out along each link, so the volume the hand
-       closes on is much further out than its joint origins suggest.
-       Measured rather than derived: with ground truth for the block and TF for the palm, a
-       block held through a carry sits at palm (0.086, 0.089, 0.002) while the frame claimed
-       (0.090, 0.050, 0.000). x and z agree to 4 mm and y is out by 39 mm, which is a frame
-       error along the closing axis and not scatter. Every finger was at or near its 1.4 N.m
-       torque clamp at the time, so the hand was gripping hard, just 39 mm too far out, where
-       the object levers itself free: it rotated from 14 to 33 degrees during the lift and slid
-       19 mm while the hand rose 184 mm.
-       It also fixes how tall an object has to be: the hand hangs 113 mm below the palm even
-       with the thumb retracted, so 28 mm below this frame, and an object shorter than that gets
-       the thumb on the table instead. See g1_manipulation's grasp_depth_below_top_m and
-       min_grip_height_m. -->
+       y = 0.050 is where the fingers and thumb meet, and it is also what fixes how tall an
+       object has to be: the hand hangs 113 mm below the palm even with the thumb retracted, so
+       63 mm below this frame, and an object shorter than that gets the thumb on the table
+       instead. See g1_manipulation's grasp_depth_below_top_m and min_grip_height_m.
+       KNOWN WRONG BY ABOUT 39 mm, and deliberately left. 0.050 is the midpoint of the thumb and
+       finger LINK ORIGINS, but their collision capsules run 50 to 62 mm out along each link, so
+       the volume the hand actually closes on is further out than the joint origins suggest.
+       Measured against ground truth: a block held through a carry sits at palm
+       (0.086, 0.089, 0.002) while this frame claims (0.090, 0.050, 0.000). x and z agree to
+       4 mm; y is out by 39 mm, along the closing axis, consistently rather than as scatter.
+       Moving it to 0.085 does seat the object properly: the block starts a carry 7 mm from the
+       frame instead of 52 to 88, and the fingers load to 0.817 N.m where they read 0.003 here.
+       It also breaks the descent. A Cartesian path is planned for THIS link, so pushing it
+       35 mm further from the wrist lengthens the lever that wrist rotation acts through, and
+       the straight line in truncates 31 to 38 % short: the pinned tabletop pick went from 3/3
+       to 0/3 across four configurations, including compensating min_grip_height_m,
+       grasp_depth_below_top_m and approach_height_m to hold the palm at the same height.
+       So the number is wrong and everything downstream is tuned around it being wrong. Fixing
+       it properly means making the descent tolerant of a frame this far out, which is the same
+       elbow-through-torso problem kinematics.yaml describes, not a one-line change. -->
   <xacro:macro name="g1_grasp_frame" params="side mirror">
     <link name="${side}_hand_grasp_frame"/>
@@ -160,5 +165,5 @@
       <parent link="${side}_hand_palm_link"/>
       <child link="${side}_hand_grasp_frame"/>
-      <origin xyz="0.090 ${mirror * 0.085} 0" rpy="0 0 0"/>
+      <origin xyz="0.090 ${mirror * 0.050} 0" rpy="0 0 0"/>
     </joint>
   </xacro:macro>

Commit message: Mount cameras from one file for the URDF and the simulator

File: workspace/src/g1_description/urdf/g1_common.xacro (robot description, xacro)
@@ -38,4 +38,43 @@
     <child link="d435_visual"/>
   </joint>
+  <!-- Cameras beyond Unitree's head D435i, mounted as config/cameras.yaml says; the simulator
+       renders them from the same file. Frames follow the relay's names for camera N: N_camera_link
+       (body), N_camera_depth_optical_frame and N_camera_color_optical_frame. -->
+  <xacro:property name="camera_mounts" value="${xacro.load_yaml('../config/cameras.yaml')}"/>
+  <xacro:macro name="depth_camera" params="name">
+    <xacro:property name="mount" value="${camera_mounts[name]}"/>
+    <link name="${name}_camera_link"/>
+    <joint name="${name}_camera_joint" type="fixed">
+      <parent link="${mount['parent']}"/>
+      <child link="${name}_camera_link"/>
+      <origin xyz="${mount['xyz'][0]} ${mount['xyz'][1]} ${mount['xyz'][2]}"
+              rpy="${mount['rpy'][0]} ${mount['rpy'][1]} ${mount['rpy'][2]}"/>
+    </joint>
+    <link name="${name}_camera_depth_optical_frame"/>
+    <joint name="${name}_camera_depth_optical_joint" type="fixed">
+      <parent link="${name}_camera_link"/>
+      <child link="${name}_camera_depth_optical_frame"/>
+      <origin xyz="0 0 0" rpy="-1.5707963267948966 0 -1.5707963267948966"/>
+    </joint>
+    <link name="${name}_camera_color_optical_frame"/>
+    <joint name="${name}_camera_color_optical_joint" type="fixed">
+      <parent link="${name}_camera_link"/>
+      <child link="${name}_camera_color_optical_frame"/>
+      <origin xyz="0 0 0" rpy="-1.5707963267948966 0 -1.5707963267948966"/>
+    </joint>
+    <link name="${name}_camera_visual">
+      <visual>
+        <origin xyz="0.0043 -0.0175 0" rpy="1.5707963267948966 0 1.5707963267948966"/>
+        <geometry>
+          <mesh filename="package://realsense2_description/meshes/d435.dae"/>
+        </geometry>
+      </visual>
+    </link>
+    <joint name="${name}_camera_visual_joint" type="fixed">
+      <parent link="${name}_camera_link"/>
+      <child link="${name}_camera_visual"/>
+    </joint>
+  </xacro:macro>
+  <xacro:depth_camera name="chest"/>
   <link name="mid360_visual">
     <visual>
